File: Hardware Designs/Logic Engine - Front LED.sch (EAGLE design)
At the start: 101 parts

Commit message: updated Front LED board to current version
Parts:
- removed C14, C15, C16, C17, C18, C19, C20, C21, C22, C23, C26, C27, C28, C29, C30, C31, C41, C42, C43, C44, C45, C46, C47, C48: 0.1uF, SparkFun-Capacitors:CAP0603-CAP
- removed L41, L42, L43, L44, L45, L46, L47, L48: WS2812B, rseries:WS2812B
Connections:
- removed net N$33: L41.DO, L42.DI
- removed net N$34: L42.DO, L43.DI
- removed net N$35: L43.DO, L44.DI
- removed net N$36: L44.DO, L45.DI
- removed net N$37: L45.DO, L46.DI
- removed net N$38: L46.DO, L47.DI
- removed net N$39: L47.DO, L48.DI
- removed net N$47: L40.DO, L41.DI
- net +5V: no longer C14.1, C15.1, C16.1, C17.1, C18.1, C19.1, C20.1, C21.1, C22.1, C23.1, C26.1, C27.1, C28.1, C29.1, C30.1, C31.1, C41.1, C42.1, C43.1, C44.1, C45.1, C46.1, C47.1, C48.1, L41.VDD, L42.VDD, L43.VDD, L44.VDD, L45.VDD, L46.VDD, L47.VDD, L48.VDD
- net DOUT: now also L40.DO; no longer L48.DO
- net GND: no longer C14.2, C15.2, C16.2, C17.2, C18.2, C19.2, C20.2, C21.2, C22.2, C23.2, C26.2, C27.2, C28.2, C29.2, C30.2, C31.2, C41.2, C42.2, C43.2, C44.2, C45.2, C46.2, C47.2, C48.2, L41.GND, L42.GND, L43.GND, L44.GND, L45.GND, L46.GND, L47.GND, L48.GND
Other:
- note added: "LEDs are not positioned like this on the board; they're in a serpentine configuration. Also, capacitors shown aren't necessarily position right next to the LED shown. My bad!"
- note added: "Please pardon the mess!"
- moved on the sheet: C10, C11, C12, C13

Commit message: Revised Front LED board slightly
Front LED board had it's mounting holes & pin headers moved down 0.04
inches. When mounting in dome this should give a little extra clearance
(0.08 inches) between the front boards.
Other:
- note removed: "LEDs are not positioned like this on the board; they're in a serpentine configuration. Also, capacitors shown aren't necessarily position right next to the LED shown. My bad!"
- note removed: "Please pardon the mess!"
Changed lines of the file:
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@@
 <sheet>
 <plain>
-<text x="-63.5" y="363.22" size="25.4" layer="91">Please pardon the mess!</text>
-<text x="134.62" y="335.28" size="8.89" layer="91" align="center">LEDs are not positioned like this on the board; they're in a serpentine configuration.
-Also, capacitors shown aren't necessarily position right next to the LED shown.
-My bad!</text>
 </plain>
 <instances>
@@
 </schematic>
 </drawing>
-<compatibility>
-<note version="6.3" minversion="6.2.2" severity="warning">
-Since Version 6.2.2 text objects can contain more than one line,
-which will not be processed correctly with this version.
-</note>
-</compatibility>
 </eagle>
