File: Hardware Designs/Teeces PSI.brd (EAGLE design)
At the start: 47.8 x 47.8 mm, 34 parts, among them IC2 MAX7219CNG

Commit message: updated Teeces PSI board design
Moved signal routing away from board edge
Parts:
- C5, C6: device SparkFun-Capacitors:CPOL-RADIAL-10UF-25V -> rseries:E2,5-5
- IN, OUT: device SparkFun-Connectors:1X05 -> rseries:1X05
- turned C5 to 180 degrees
- turned C6 to 180 degrees
Connections:
- net +5V: now also C5.+, C6.+; no longer C5.1, C6.1
- net GND: now also C5.-, C6.-; no longer C5.2, C6.2
Routing:
- net +5V: track 0.00 -> 82.0 mm, vias 0 -> 2
- net GND: track 0.00 -> 75.3 mm, vias 0 -> 2
- net LOAD: track 80.3 -> 52.2 mm, vias 1 -> 0
- net DIN: track 66.5 -> 51.6 mm
- net DOUT: track 47.8 -> 40.6 mm
- net SEGDP: track 72.5 -> 65.5 mm, vias 1 -> 0
- net SEGB: track 40.9 -> 45.9 mm
- net DIG4: track 38.9 -> 36.2 mm, vias 2 -> 0
- net DIG0: track 40.7 -> 39.5 mm
- net DIG2: track 35.8 -> 34.7 mm
- net DIG5: track 26.1 -> 26.6 mm, vias 2 -> 1
- net CLK: track 51.0 -> 50.9 mm, vias 2 -> 1
- removed copper zone on layer 1, net +5V
- removed copper zone on layer 16, net GND
Other:
- board text added: "Paul Murphy 2020"
- board text added: "TEECES PSI 3.5"
- board text removed: "TEECES PSI 3.3"
