File: Hardware Designs/Teeces PSI.sch (EAGLE design)
At the start: 34 parts, among them IC2 MAX7219CNG

Commit message: updated Teeces PSI board design
Moved signal routing away from board edge
Parts:
- C5, C6: device SparkFun-Capacitors:10UF-25V-20%(PTH) -> rseries:CPOL-USE2.5-5
- IN, OUT: device SparkFun-Connectors:M05PTH -> rseries:CONN_05
